File: flat.sch (EAGLE design)
At the start: 76 parts

Commit message: finished first version
Parts:
- added JP35: (no value), SparkFun-Connectors:M02-JST-2-PTH-NO_SILK
- added P13: (no value), e-lampen-signalisation:SIGNALLAMPE
- added SP1: SPEAKER/AL11P, adafruit:SPEAKER/AL11P
Other:
- note added: "10"
- note added: "10A"
- note added: "11"
- note added: "16A"
- note added: "25A"
- note added: "3"
- note added: "4"
- note added: "6"
- note added: "7"
- note added: "9"
- moved on the sheet: P4, S15

Commit message: update after the flat renovation 2015
Parts:
- removed JP34: (no value), SparkFun-Connectors:M02-JST-2-PTH-NO_SILK
Other:
- note added: "Boiler"
Changed lines of the file:
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@@
 <part name="JP32" library="SparkFun-Connectors" deviceset="M02" device="-JST-2-PTH-NO_SILK"/>
 <part name="JP33" library="SparkFun-Connectors" deviceset="M02" device="-JST-2-PTH-NO_SILK"/>
-<part name="JP34" library="SparkFun-Connectors" deviceset="M02" device="-JST-2-PTH-NO_SILK"/>
 <part name="S3" library="adafruit" deviceset="31-XX" device=""/>
 <part name="S4" library="adafruit" deviceset="31-XX" device=""/>
@@
 <text x="-22.86" y="284.48" size="5.08" layer="97">16A</text>
 <text x="190.5" y="330.2" size="5.08" layer="97">10A</text>
+<text x="388.62" y="327.66" size="6.4516" layer="97" ratio="9">Boiler</text>
 </plain>
 <instances>
@@
 <instance part="JP32" gate="G$1" x="433.88" y="28" rot="R180"/>
 <instance part="JP33" gate="G$1" x="498" y="146.12" rot="R90"/>
-<instance part="JP34" gate="G$1" x="448" y="146.12" rot="R90"/>
 <instance part="S3" gate="1" x="103.5" y="162.86"/>
 <instance part="S4" gate="1" x="113.5" y="162.86"/>
@@
 <bus name="B$21">
 <segment>
-<wire x1="444.5" y1="175.26" x2="541.02" y2="175.26" width="0.762" layer="92"/>
+<wire x1="444.5" y1="175.26" x2="495.3" y2="175.26" width="0.762" layer="92"/>
+<wire x1="495.3" y1="175.26" x2="541.02" y2="175.26" width="0.762" layer="92"/>
 <wire x1="541.02" y1="175.26" x2="541.02" y2="162.56" width="0.762" layer="92"/>
 <wire x1="541.02" y1="162.56" x2="586.74" y2="162.56" width="0.762" layer="92"/>
 <wire x1="586.74" y1="162.56" x2="586.74" y2="299.72" width="0.762" layer="92"/>
 <wire x1="586.74" y1="299.72" x2="487.68" y2="299.72" width="0.762" layer="92"/>
-</segment>
-</bus>
+<wire x1="495.3" y1="154.94" x2="495.3" y2="175.26" width="0.762" layer="92"/>
+</segment>
+</bus>
