File: dubnov_kitchen_box.sch (EAGLE design)
At the start: 0 parts

Commit message: Dubnov kitchen design rc1
Other:
- note added: "Box (2pcs)"
- note added: "Furniture: Hinges Blum: Half overlay regular 16 pcs 180 degrees 8 pcs Handles 8 pcs"
- note added: "Wood bars 65.0 x 5.0 x 2.8 - 2 pcs 53.0 x 5.0 x 2.0 - 2 pcs"
- note removed: "Bottom"
- note removed: "Top"
Changed lines of the file:
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@@
 <?xml version="1.0" encoding="utf-8"?>
 <!DOCTYPE eagle SYSTEM "eagle.dtd">
-<eagle version="7.3.0">
+<eagle version="7.6.0">
 <drawing>
 <settings>
@@
 <wire x1="27.8" y1="40" x2="1" y2="40" width="0.3048" layer="94"/>
 <wire x1="1" y1="40" x2="1" y2="1" width="0.3048" layer="94"/>
-<wire x1="-0.95" y1="0" x2="-0.95" y2="-2" width="0.3048" layer="94"/>
-<wire x1="-0.95" y1="-2" x2="29.75" y2="-2" width="0.3048" layer="94"/>
-<wire x1="29.75" y1="-2" x2="29.75" y2="0" width="0.3048" layer="94"/>
-<wire x1="29.75" y1="0" x2="28.8" y2="0" width="0.3048" layer="94"/>
-<wire x1="-0.95" y1="0" x2="0" y2="0" width="0.3048" layer="94"/>
 <dimension x1="28.8" y1="41" x2="0" y2="41" x3="14.4" y3="46" textsize="1.778" layer="97" precision="1"/>
 <dimension x1="28.8" y1="0" x2="28.8" y2="41" x3="37" y3="20.5" textsize="1.778" layer="97" precision="1"/>
-<dimension x1="-0.95" y1="-2" x2="29.75" y2="-2" x3="14.4" y3="-11" textsize="1.778" layer="97" precision="1"/>
 <wire x1="50" y1="0" x2="59" y2="0" width="0.3048" layer="94"/>
 <wire x1="59" y1="0" x2="59" y2="41" width="0.3048" layer="94"/>
 <wire x1="59" y1="41" x2="50" y2="41" width="0.3048" layer="94"/>
 <wire x1="50" y1="41" x2="50" y2="0" width="0.3048" layer="94"/>
-<wire x1="50" y1="0" x2="49.5" y2="0" width="0.3048" layer="94"/>
-<wire x1="49.5" y1="0" x2="49.5" y2="-2" width="0.3048" layer="94"/>
-<wire x1="49.5" y1="-2" x2="59.7" y2="-2" width="0.3048" layer="94"/>
-<wire x1="59.7" y1="-2" x2="59.7" y2="0" width="0.3048" layer="94"/>
-<wire x1="59.7" y1="0" x2="59" y2="0" width="0.3048" layer="94"/>
-<dimension x1="49.5" y1="-2" x2="59.7" y2="-2" x3="54.6" y3="-11" textsize="1.778" layer="97" precision="1"/>
 <dimension x1="59" y1="41" x2="50" y2="41" x3="54.5" y3="46" textsize="1.778" layer="97" precision="1"/>
-<dimension x1="59.7" y1="0" x2="59" y2="0" x3="59.35" y3="7" textsize="1.778" layer="97" precision="1"/>
-<dimension x1="50" y1="0" x2="49.5" y2="0" x3="49.75" y3="4" textsize="1.778" layer="97" dtype="horizontal" precision="1"/>
-<text x="62" y="16" size="1.778" layer="97" rot="R90">Top</text>
-<text x="49" y="15" size="1.778" layer="97" rot="R90">Bottom</text>
+<text x="21" y="57" size="2.54" layer="97">Box (2pcs)</text>
+<text x="78" y="42" size="2.54" layer="97">Wood bars
+65.0 x 5.0 x 2.8 - 2 pcs
+53.0 x 5.0 x 2.0 - 2 pcs</text>
+<text x="78" y="2" size="2.54" layer="97">Furniture:
+Hinges Blum:
+Half overlay regular  16 pcs
+180 degrees              8 pcs
+Handles                     8 pcs</text>
 </plain>
 <instances>
@@
 </schematic>
 </drawing>
+<compatibility>
+<note version="6.3" minversion="6.2.2" severity="warning">
+Since Version 6.2.2 text objects can contain more than one line,
+which will not be processed correctly with this version.
+</note>
+</compatibility>
 </eagle>
